Commit message: Fix idle drift velocity

File: my_rb1_description/urdf/my_rb1_robot.urdf (robot description, URDF)
Before this commit: robot my_rb1_robot, 7 links, 6 joints
Links:
- removed link back_caster
- removed link base_footprint
- removed link base_link
- removed link front_caster
- removed link front_laser
- removed link left_wheel
- removed link right_wheel
Joints:
- removed joint base_footprint_to_base_link
- removed joint joint_base_link_back_caster
- removed joint joint_base_link_front_caster
- removed joint joint_base_link_front_laser
- removed joint joint_base_link_left_wheel
- removed joint joint_base_link_right_wheel

Commit message: Restore deleted code

File: my_rb1_description/urdf/my_rb1_robot.urdf (robot description, URDF)
Before this commit: robot my_rb1_robot, 0 links, 0 joints
Links:
- added link back_caster, mass 1; collision sphere radius=0.025; visual sphere radius=0.025
- added link base_footprint
- added link base_link, mass 20; collision cylinder length=0.3 radius=0.25; visual cylinder length=0.3 radius=0.25
- added link front_caster, mass 1; collision sphere radius=0.025; visual sphere radius=0.025
- added link front_laser, mass 1; collision cylinder length=0.04 radius=0.04; visual cylinder length=0.04 radius=0.04
- added link left_wheel, mass 1; collision cylinder length=0.05 radius=0.025; visual cylinder length=0.05 radius=0.025
- added link right_wheel, mass 1; collision cylinder length=0.05 radius=0.025; visual cylinder length=0.05 radius=0.025
Joints:
- added joint base_footprint_to_base_link: type fixed, parent base_footprint, child base_link, origin xyz=0 0 0.15 rpy=0 0 0
- added joint joint_base_link_back_caster: type fixed, parent base_link, child back_caster, origin xyz=-0.1 0.0 -0.15 rpy=0 0 0
- added joint joint_base_link_front_caster: type fixed, parent base_link, child front_caster, origin xyz=0.1 0.0 -0.15 rpy=0 0 0
- added joint joint_base_link_front_laser: type fixed, parent base_link, child front_laser, origin xyz=0.25 0.0 0.075 rpy=3.14 0 0
- added joint joint_base_link_left_wheel: type continuous, parent base_link, child left_wheel, origin xyz=0.0 0.2 -0.15 rpy=0 0 0, axis 0 1 0, limit effort=10000 velocity=1000
- added joint joint_base_link_right_wheel: type continuous, parent base_link, child right_wheel, origin xyz=0.0 -0.2 -0.15 rpy=0 0 0, axis 0 1 0, limit effort=10000 velocity=1000
